Commit message: added excavation tasks success.

File: ravens/environments/assets/ur5/bucket/bucket.urdf (robot description, URDF)
Before this commit: robot bucket.urdf, 2 links, 1 joints
Links:
- link midLink: geometry collision mesh filename=bucket.obj scale=1 1 1; visual mesh filename=bucket/bucket.obj scale=1 1 1
